File: hw/kicad/v5.0/stmbl_5.0.kicad_pcb (KiCad board)
At the start: 2 copper layers, 99.8 x 99.8 mm, 432 parts, among them J1 RJ45_LED, J2 RJ45_LED, J3 RJ45_LED, P1 USB_C_Receptacle_USB2.0, P10 CONN_02X06, P11 USB_C_Receptacle_USB2.0, P12 CONN_01X04, P15 CONN_01X02, P2 CONN_01X02, P3 CONN_01X02, P4 CONN_01X02, P5 CONN_01X06, P6 CONN_01X02, P7 CONN_01X04, P8 CONN_01X03, P9 CONN_01X06, Q1 IRLML6344, Q2 IRLML6344, Q3 IRLML6344, Q4 IRLML6344, Q5 IRLML6344, T1 testpoint, T2 testpoint, T44 testpoint, T45 testpoint, T46 testpoint, U1 USBLC6-4SC6, U10 SN65176B, U11 SN65176B, U12 IKCM30F60GAXKMA1, U13 RT8259, U14 SN65176B, U15 SN65176B, U16 SN65176B, U17 SN65176B, U18 SN65176B, U19 SN65176B, U2 zldo1117, U20 USBLC6-4SC6, U21 USBLC6-4SC6, U22 USBLC6-4SC6, U23 USBLC6-4SC6, U234 fan, U24 RT8259, U25 STM32F303CBTx, U26 STM32F405VG, U28 RT8259, U29 USBLC6-4SC6, U3 SI8621, U4 RT8259, U5 LNK304D, U6 LM358, U7 LM358, U8 SN65176B, U9 SN65176B, Y1 8M, Y2 8M

Commit message: JLCPCB production files
Parts:
- added REF**: JLC_Tooling_Hole, v5:JLC_Tooling_Hole, F.Cu at (196.5, 148.0)
- added REF**: JLC_Tooling_Hole, v5:JLC_Tooling_Hole, F.Cu at (107.5, 53.5)
- added REF**: JLC_Tooling_Hole, v5:JLC_Tooling_Hole, F.Cu at (107.5, 148.0)
- moved G*** 16.2 mm to (156.0, 102.5)
- moved G*** 5.50 mm to (176.0, 114.5)
- moved LOGO2 0.70 mm to (183.8, 141.7)
- moved C17 0.10 mm to (192.8, 53.6)
Routing:
- net /ctrl/FB0/D45: track 61.7 -> 50.1 mm
- net /ctrl/CMD/D45: track 70.9 -> 69.6 mm
- net +24V: vias 15 -> 13
Other:
- board text added: "JLCJLCJLCJLC"
- board text added: "STMBL 5.0; JLC by jst"
- board text added: "https://github.com/freakontrol/stmbl https://github.com/jstjst/stmbl"
- board text removed: "STMBL 5.0"
- board text removed: "https://github.com/freakontrol/stmbl"
